Commit message: 4-1: add collision

File: install/my_robot_description/share/my_robot_description/urdf/arm.xacro (robot description, xacro)
@@ -9,4 +9,10 @@
       <material name="gray"/>
     </visual>
+    <collision>
+      <geometry>
+        <box size="0.4 0.4 0.1"/>
+      </geometry>
+      <origin xyz="0.0 0.0 0.05" rpy="0.0 0.0 0.0"/>
+    </collision>
   </link>
   <joint name="joint1" type="revolute">
@@ -25,4 +31,10 @@
       <material name="blue"/>
     </visual>
+    <collision>
+      <geometry>
+        <cylinder length="0.5" radius="0.1"/>
+      </geometry>
+      <origin xyz="0.0 0.0 0.25" rpy="0.0 0.0 0.0"/>
+    </collision>
   </link>
   <joint name="joint2" type="revolute">
@@ -41,4 +53,10 @@
       <material name="gray"/>
     </visual>
+    <collision>
+      <geometry>
+        <cylinder length="0.6" radius="0.05"/>
+      </geometry>
+      <origin xyz="0.0 0.0 0.3" rpy="0.0 0.0 0.0"/>
+    </collision>
   </link>
   <joint name="joint3" type="revolute">
@@ -57,4 +75,10 @@
       <material name="blue"/>
     </visual>
+    <collision>
+      <geometry>
+        <cylinder length="0.1" radius="0.05"/>
+      </geometry>
+      <origin xyz="0.0 0.0 0.05" rpy="0.0 0.0 0.0"/>
+    </collision>
   </link>
   <joint name="joint4" type="revolute">
@@ -73,4 +97,10 @@
       <material name="gray"/>
     </visual>
+    <collision>
+      <geometry>
+        <cylinder length="0.5" radius="0.05"/>
+      </geometry>
+      <origin xyz="0.0 0.0 0.25" rpy="0.0 0.0 0.0"/>
+    </collision>
   </link>
   <joint name="joint5" type="revolute">
@@ -89,4 +119,10 @@
       <material name="blue"/>
     </visual>
+    <collision>
+      <geometry>
+        <box size="0.1 0.1 0.05"/>
+      </geometry>
+      <origin xyz="0.0 0.0 0.025" rpy="0.0 0.0 0.0"/>
+    </collision>
   </link>
    <joint name="joint6" type="continuous">
@@ -104,4 +140,10 @@
       <material name="gray"/>
     </visual>
+    <collision>
+      <geometry>
+        <box size="0.1 0.1 0.02"/>
+      </geometry>
+      <origin xyz="0.0 0.0 0.01" rpy="0.0 0.0 0.0"/>
+    </collision>
   </link>
   <joint name="hand_tool_joint" type="fixed">

Commit message: chapter4: moveit setup assistant

File: install/my_robot_description/share/my_robot_description/urdf/arm.xacro (robot description, xacro)
@@ -22,4 +22,5 @@
     <axis xyz="0.0 0.0 1.0"/>
     <limit lower="-3.14" upper="3.14" effort="1000.0" velocity="1.0"/>
+    <safety_controller k_position="100.0" k_velocity="10.0" soft_lower_limit="-3.14" soft_upper_limit="3.14"/>
   </joint>
   <link name="shoulder_link">
@@ -44,4 +45,5 @@
     <axis xyz="0.0 1.0 0.0"/>
     <limit lower="0" upper="2.5" effort="1000.0" velocity="1.0"/>
+    <safety_controller k_position="100.0" k_velocity="10.0" soft_lower_limit="0" soft_upper_limit="2.5"/>
   </joint>
   <link name="arm_link">
@@ -66,4 +68,5 @@
     <axis xyz="0.0 1.0 0.0"/>
     <limit lower="0" upper="2.5" effort="1000.0" velocity="1.0"/>
+    <safety_controller k_position="100.0" k_velocity="10.0" soft_lower_limit="0" soft_upper_limit="2.5"/>
   </joint>
   <link name="elbow_link">
@@ -88,4 +91,5 @@
     <axis xyz="0.0 0.0 1.0"/>
     <limit lower="-3.14" upper="3.14" effort="1000.0" velocity="1.0"/>
+    <safety_controller k_position="100.0" k_velocity="10.0" soft_lower_limit="-3.14" soft_upper_limit="3.14"/>
   </joint>
   <link name="forearm_link">
@@ -110,4 +114,5 @@
     <axis xyz="0.0 1.0 0.0"/>
     <limit lower="0" upper="2.5" effort="1000.0" velocity="1.0"/>
+    <safety_controller k_position="100.0" k_velocity="10.0" soft_lower_limit="0" soft_upper_limit="2.5"/>
   </joint>
   <link name="wrist_link">
@@ -131,4 +136,6 @@
     <origin xyz="0.0 0.0 0.05" rpy="0.0 0.0 0.0"/>
     <axis xyz="0.0 0.0 1.0"/>
+    <limit lower="-3.14" upper="3.14" effort="1000.0" velocity="1.0"/>
+    <safety_controller k_position="100.0" k_velocity="10.0" soft_lower_limit="-3.14" soft_upper_limit="3.14"/>
   </joint>
   <link name="hand_link">

Commit message: modify

File: install/my_robot_description/share/my_robot_description/urdf/arm.xacro (robot description, xacro)
@@ -34,5 +34,5 @@
     <collision>
       <geometry>
-        <cylinder length="0.5" radius="0.1"/>
+        <box size="0.2 0.2 0.5"/>
       </geometry>
       <origin xyz="0.0 0.0 0.25" rpy="0.0 0.0 0.0"/>
@@ -57,5 +57,5 @@
     <collision>
       <geometry>
-        <cylinder length="0.6" radius="0.05"/>
+        <box size="0.1 0.1 0.6"/>
       </geometry>
       <origin xyz="0.0 0.0 0.3" rpy="0.0 0.0 0.0"/>
@@ -80,5 +80,5 @@
     <collision>
       <geometry>
-        <cylinder length="0.1" radius="0.05"/>
+        <box size="0.1 0.1 0.1"/>
       </geometry>
       <origin xyz="0.0 0.0 0.05" rpy="0.0 0.0 0.0"/>
@@ -103,5 +103,5 @@
     <collision>
       <geometry>
-        <cylinder length="0.5" radius="0.05"/>
+        <box size="0.1 0.1 0.5"/>
       </geometry>
       <origin xyz="0.0 0.0 0.25" rpy="0.0 0.0 0.0"/>
