Commit message: connect the gripper

File: install/my_robot_description/share/my_robot_description/urdf/common_properties.xacro (robot description, xacro)
@@ -7,3 +7,9 @@
       <color rgba="0.0 0.0 0.5 1"/>
   </material>
+  <material name="dark_green">
+      <color rgba="0.0 0.5 0.0 1"/>
+  </material>
+  <material name="light_green">
+      <color rgba="0.0 1.0 0.0 1"/>
+  </material>
 </robot>

File: install/my_robot_description/share/my_robot_description/urdf/my_robot_urdf.xacro (robot description, xacro)
@@ -3,3 +3,9 @@
   <xacro:include filename="common_properties.xacro"/>
   <xacro:include filename="arm.xacro"/>
+  <xacro:include filename="gripper.xacro"/>
+  <joint name="gripper_base_joint" type="fixed">
+      <parent link="tool_link" />
+      <child link="gripper_base_link" />
+      <origin xyz="0 0 0" rpy="0 0 0" />
+  </joint>
 </robot>

File: install/my_robot_moveit_config/share/my_robot_moveit_config/config/my_robot.urdf.xacro (robot description, xacro)
@@ -3,5 +3,5 @@
     <xacro:arg name="initial_positions_file" default="initial_positions.yaml" />
     <!-- Import my_robot urdf file -->
-    <xacro:include filename="$(find my_robot_description)/urdf/my_robot.urdf.xacro" />
+    <xacro:include filename="$(find my_robot_description)/urdf/my_robot_urdf.xacro" />
     <!-- Import control_xacro -->
     <xacro:include filename="my_robot.ros2_control.xacro" />
